Commit message: ROS 2 Humble stack: driver fixes, MowgliNext GUI integration, bringup, Nav2, deploy tooling
- Drivers: bumper_controller compiles (PID members, delegating ctor, typed service cb) and
  publishes Twist on /cmd_vel_bumper; WIT IMU rewritten for the 11-byte WIT protocol and
  publishes /imu/data; gps_gate + um960 use Humble NavSatStatus values (RTK -> GBAS_FIX,
  DGPS -> SBAS_FIX); MCU driver gains /cutter_control, /charging, /clear_estop, /cutter_off,
  /mower_base/status, /estop, lift/stop interlocks, e-stop latch, cutter-off on shutdown,
  9-element IMU covariances; /cmd_vel is unstamped Twist (+ /cmd_vel_stamped).
- Command chain: twist_mux lanes (nav 10, docking 15, teleop 20, bumper 50, emergency 100,
  /estop lock) -> /cmd_vel_raw -> cmd_vel_slew -> /cmd_vel. base_ble on /cmd_vel_teleop.
- New packages: mower_teleop (ws relay + mux config), mower_gui_bridge (MowgliNext GUI
  adapter + stub high-level state machine), mower_bringup (mower.launch.py entry point),
  mower_navigation (Humble Nav2 params, all lifecycle nodes activate), mowgli_interfaces
  (vendored, GPL-3.0).
- mower_coverage: Fields2Cover 2.1 API fixes, swath trimming to the drivable region,
  angle bugs; 15/15 gtests. mower_proto regenerated for protobuf 3.12.
- Localization: ekf.yaml float covariances, datum_lat/lon/yaw launch args pin the map
  origin, static map->odom for Phase A, URDF base_footprint + blade_link.
- Tests pass on the host (stubs) and under real rclpy (colcon test: 188 tests, 0 failures).
- Docker: amd64 dev image + scripts/dev_build.sh, Dockerfile.humble deps (pip websockets:
  Jammy apt 9.1 is broken on py3.10), compose runs the launch, GUI image (gui/Dockerfile,
  arm64 cross-build), docker-compose.gui.yml, scripts/deploy_to_mower.sh.
- third_party/mowglinext: GUI + reference packages (COLCON_IGNORE), Tron feature flags.
- docs: STATUS.md, audit_2026-10-05/, gui.md.

File: config/urdf/mower.urdf.xacro (robot description, xacro)
@@ -7,5 +7,6 @@
   same model with per-chassis mounting offsets — adjust the properties
   below to match a specific unit).
-  Loaded by the robot_state_publisher entry in launch/nav2.launch.py:
+  Loaded by the robot_state_publisher in launch/mower.launch.py (and
+  launch/nav2.launch.py when run standalone):
       robot_description = xacro <stack_root>/config/urdf/mower.urdf.xacro
   ======================================================================
@@ -48,4 +49,12 @@
               Front stereo (Metoak). No driver ported yet — planned
               stereo_vio_bridge; frame reserved here.
+  base_footprint
+              Identity child of base_link (fixed joint). MowgliNext nodes
+              (e.g. mowgli_map map_server_node) look up
+              map -> base_footprint, so the frame must exist. Planar
+              robot: no ground-projection offset is needed today.
+  blade_link  Alias of cutter_link (same origin: the cutter disc
+              centre), the frame name MowgliNext coverage/mowing code
+              expects. Fixed joint from base_link.
   cutter_link, left/right_wheel, left/right_omni_wheel
               Geometry/visualization only. The MCU owns the cutter
@@ -169,4 +178,19 @@
     <origin xyz="${cutter_xyz}" rpy="0 0 0"/>
   </joint>
+  <!-- blade_link: MowgliNext name for the cutter disc centre. Same origin
+       as cutter_link (kept for existing consumers). -->
+  <link name="blade_link"/>
+  <joint name="blade_joint" type="fixed">
+    <parent link="base_link"/>
+    <child link="blade_link"/>
+    <origin xyz="${cutter_xyz}" rpy="0 0 0"/>
+  </joint>
+  <!-- base_footprint: identity child of base_link (MowgliNext requires it). -->
+  <link name="base_footprint"/>
+  <joint name="base_footprint_joint" type="fixed">
+    <parent link="base_link"/>
+    <child link="base_footprint"/>
+    <origin xyz="0 0 0" rpy="0 0 0"/>
+  </joint>
   <xacro:drive_wheel side="left"  y_sign="-1"/>
   <xacro:drive_wheel side="right" y_sign="1"/>

Commit message: Stack: set_datum (bridge writes datum.env + GUI yaml, calls /datum), EKF config fix (no double absolute pose, yaw rate slot), cut_width/swath_overlap args, blade_link visual, correction_stream mirror, low-CPU subscription pump across Python nodes, lights/base_keys, web_video_server on by default, mediamtx QoS, fastdds shm clean at start

File: config/urdf/mower.urdf.xacro (robot description, xacro)
@@ -95,4 +95,8 @@
   <xacro:property name="bumper_xyz" value="0.50718 0 0"/>
   <xacro:property name="cutter_xyz" value="0.3 0 -0.05"/>
+  <!-- Cutter disc radius: 0.20 m cut width. TODO: measure the blade tip circle on the
+       Tron and update this, the coverage cut_width_m launch arg (mower.launch.py) and
+       mower_coverage's default together. -->
+  <xacro:property name="cutter_radius" value="0.10"/>
   <!-- Camera mounts (vendor values). -->
   <xacro:property name="stereo_cam_xyz" value="0.466 0 0.25"/>
@@ -168,5 +172,5 @@
     <visual>
       <geometry>
-        <cylinder radius="0.1" length="0.05"/>
+        <cylinder radius="${cutter_radius}" length="0.05"/>
       </geometry>
       <material name="red"/>
@@ -179,6 +183,15 @@
   </joint>
   <!-- blade_link: MowgliNext name for the cutter disc centre. Same origin
-       as cutter_link (kept for existing consumers). -->
-  <link name="blade_link"/>
+       as cutter_link (kept for existing consumers). Its visual is the blade
+       disc itself (true radius, thin): the GUI draws the blade silhouette
+       from this cylinder. -->
+  <link name="blade_link">
+    <visual>
+      <geometry>
+        <cylinder radius="${cutter_radius}" length="0.004"/>
+      </geometry>
+      <material name="red"/>
+    </visual>
+  </link>
   <joint name="blade_joint" type="fixed">
     <parent link="base_link"/>

Commit message: Front stereo hardware depth into Nav2: stereo_depth node decodes /dev/video11 RGBD frames to PointCloud2; local costmap obstacle source; stereo_camera_optical frame

File: config/urdf/mower.urdf.xacro (robot description, xacro)
@@ -223,4 +223,14 @@
   <xacro:box_sensor name="stereo_camera" xyz="${stereo_cam_xyz}"
                     rpy="1.64061 0 1.57079" size="${sensor_box}" material="yellow"/>
+  <!-- Optical frame of the Metoak hardware disparity (mower_cameras/stereo_depth, ~/points):
+       standard optical axes (z forward, x right, y down). Pose from a floor-plane fit of the
+       live depth cloud on 2026-10-06 (best fit: no pitch, 0.215 m above base_link/ground);
+       the stereo_camera box above keeps the vendor pose. Re-fit after any mount change. -->
+  <link name="stereo_camera_optical"/>
+  <joint name="stereo_camera_optical_joint" type="fixed">
+    <parent link="base_link"/>
+    <child link="stereo_camera_optical"/>
+    <origin xyz="0.466 0 0.215" rpy="-1.5707963 0 -1.5707963"/>
+  </joint>
   <!-- OA cameras — frames match cameras.launch.py camera_frame_id. -->
   <xacro:box_sensor name="left_oa_camera" xyz="${oa_cam_xyz}"

Commit message: Stereo costmap: measured camera pose, speckle/ground-plane/persistence filters, stereo source tuning, stereo_costmap:=false switch; stereo_cam per-eye conversion; det_range fallback pose; nav params test for PathProgressGoalChecker

File: config/urdf/mower.urdf.xacro (robot description, xacro)
@@ -224,12 +224,17 @@
                     rpy="1.64061 0 1.57079" size="${sensor_box}" material="yellow"/>
   <!-- Optical frame of the Metoak hardware disparity (mower_cameras/stereo_depth, ~/points):
-       standard optical axes (z forward, x right, y down). Pose from a floor-plane fit of the
-       live depth cloud on 2026-10-06 (best fit: no pitch, 0.215 m above base_link/ground);
-       the stereo_camera box above keeps the vendor pose. Re-fit after any mount change. -->
+       standard optical axes (z forward, x right, y down). MEASURED from the depth ground plane
+       on 2026-10-06 (robot at the dock on flat lawn, 10 s / 79 frames of /stereo_depth/points,
+       RANSAC + least-squares plane over 0.4-2.2 m, 115k inliers, residual 9 mm):
+       camera 0.240 m above the ground, pitched UP 0.92 deg, roll 0.03 deg (ignored).
+       The earlier fit (0.215 m, no pitch) put the lawn at -0.02..-0.05 m sinking with range.
+       rpy: pitch-up about base y folds into the optical roll term (-pi/2 + 0.01600).
+       The stereo_camera box above keeps the vendor pose. Re-measure after any mount change
+       (stereo_depth publishes the live fit on /stereo_depth/ground_plane). -->
   <link name="stereo_camera_optical"/>
   <joint name="stereo_camera_optical_joint" type="fixed">
     <parent link="base_link"/>
     <child link="stereo_camera_optical"/>
-    <origin xyz="0.466 0 0.215" rpy="-1.5707963 0 -1.5707963"/>
+    <origin xyz="0.466 0 0.240" rpy="-1.5547956 0 -1.5707963"/>
   </joint>
   <!-- OA cameras — frames match cameras.launch.py camera_frame_id. -->

Commit message: Stereo: synchronised 10 Hz mono8 pair from one buffer (DDS rmem cap was the loss), colour right eye on demand for YOLO; Metoak ICM-42600 IMU via kernel IIO at 200 Hz (/stereo_imu/data) with batch re-stamping and bias; VIO metoak config + lever-arm removal; setup_stereo_host.sh

File: config/urdf/mower.urdf.xacro (robot description, xacro)
@@ -238,4 +238,18 @@
     <origin xyz="0.466 0 0.240" rpy="-1.5547956 0 -1.5707963"/>
   </joint>
+  <!-- Metoak stereo IMU (ICM-40608 on i2c 8-0068; mower_cameras/stereo_imu -> /stereo_imu/data,
+       frame stereo_camera_imu = the chip's own axes). Factory IMU<->cam0 extrinsic from the vendor
+       VIO configs (src/mower_localization/vision_localization/config/metoak/sn*_euroc_stereo_imu.yaml,
+       body_T_cam0 = [R=diag(-1,1,-1) | p_CinI=(0.05143, -0.00453, -0.01503)], a mechanical constant)
+       inverted to the IMU pose in the camera optical frame: p_IinC = (0.05143, 0.00453, -0.01503),
+       R = Ry(pi). Assumes stereo_camera_optical ~ cam0 (the disparity reference eye; eye order is
+       still to be confirmed, docs/vio.md 3.6). Checked at rest 2026-10-07: accel (-0.03, -9.79,
+       +0.32) m/s^2, i.e. IMU y = camera y (down) and IMU z = -camera z, as this rotation predicts. -->
+  <link name="stereo_camera_imu"/>
+  <joint name="stereo_camera_imu_joint" type="fixed">
+    <parent link="stereo_camera_optical"/>
+    <child link="stereo_camera_imu"/>
+    <origin xyz="0.05143 0.00453 -0.01503" rpy="0 3.14159265 0"/>
+  </joint>
   <!-- OA cameras — frames match cameras.launch.py camera_frame_id. -->
   <xacro:box_sensor name="left_oa_camera" xyz="${oa_cam_xyz}"

Commit message: localization: GNSS antenna lever arm x 0.10 m (URDF gps_link), mirrored in mower_sim
The owner measured the antenna centre 0.10 m ahead of the rear axle, centred. The URDF
had gps_link at (0, 0, 0.3), so navsat_transform put base_link at the antenna: the field
pivot test saw a 7-10 cm /fix circle and 0.08-0.19 m of EKF displacement per pivot while
the axle stayed put. UM960 stamps frame_id gps_link (bringup.launch.py), so the URDF is
the one place to change. mower_sim's /fix is now the antenna (gps_antenna_x/_y, a test
keeps them equal to the URDF).

File: config/urdf/mower.urdf.xacro (robot description, xacro)
@@ -37,5 +37,11 @@
               arm — without it, it silently assumes the receiver sits
               at the robot origin.
-              TODO(calib): antenna mounting offset (vendor: z=+0.30).
+              Offset: x +0.10 measured by the owner 2026-10-20 (antenna
+              centre 0.10 m ahead of the rear axle, centred left-right);
+              z +0.30 vendor. Before it was (0, 0, 0.3) and navsat put
+              base_link at the antenna: the field pivot test saw a 7-10 cm
+              /fix circle and 0.08-0.19 m of EKF "displacement" per pivot
+              with the axle still (docs/analysis/2026-10-20_error_budget.md).
+              mower_sim's gps_antenna_x/_y mirror this (test_world checks).
   bumper      Bumper strip geometry. mower_mcu_driver reports bumper
               state in MowerSensorInfo (bumper / bumper_l / bumper_r
@@ -92,5 +98,5 @@
        identity broadcast (see the frame contract above). -->
   <xacro:property name="imu_xyz"    value="0 0 0"/>
-  <xacro:property name="gps_xyz"    value="0 0 0.3"/>
+  <xacro:property name="gps_xyz"    value="0.10 0 0.3"/>
   <xacro:property name="bumper_xyz" value="0.50718 0 0"/>
   <xacro:property name="cutter_xyz" value="0.3 0 -0.05"/>
@@ -214,5 +220,5 @@
        broadcast (see frame contract). TODO(calib): real offset here. -->
   <xacro:box_sensor name="imu_link" xyz="${imu_xyz}" rpy="0 0 0" size="${sensor_box}" material="green"/>
-  <!-- GNSS antenna (UM960). TODO(calib): real lever arm here. -->
+  <!-- GNSS antenna (UM960): measured lever arm (x 0.10, owner 2026-10-20). -->
   <xacro:box_sensor name="gps_link" xyz="${gps_xyz}" rpy="0 0 0" size="${sensor_box}" material="red"/>
   <!-- Bumper strip. -->

Commit message: urdf: cutter/blade_link at the measured deck centre x 0.25 (was 0.3); map_server fallback 0.25
The owner measured the cutting deck centre 0.25 m ahead of the rear axle, centred.
blade_link (map_server mow progress) and cutter_link share cutter_xyz; the map_server
blade_offset_x fallback now agrees (test_world checks both).

File: config/urdf/mower.urdf.xacro (robot description, xacro)
@@ -100,5 +100,8 @@
   <xacro:property name="gps_xyz"    value="0.10 0 0.3"/>
   <xacro:property name="bumper_xyz" value="0.50718 0 0"/>
-  <xacro:property name="cutter_xyz" value="0.3 0 -0.05"/>
+  <!-- cutter_xyz x 0.25 (was 0.3): the owner measured the deck centre 0.25 m ahead of the
+       rear axle, centred (2026-10-20). cutter_link and blade_link share it; map_server's mow
+       progress looks up base_link -> blade_link (fallback blade_offset_x, also 0.25). -->
+  <xacro:property name="cutter_xyz" value="0.25 0 -0.05"/>
   <!-- Cutter disc radius: 0.20 m cut width. TODO: measure the blade tip circle on the
        Tron and update this, the coverage cut_width_m launch arg (mower.launch.py) and

Commit message: urdf: owner/vendor geometry - gps_link (0.098, 0, 0.214), blade/cutter x 0.23, stereo optical y -0.041
gps_link: vendor ESKF base_gps_x 0.098 (CAD; owner measured 0.10), antenna top 0.214 m above
the axle. Deck centre exactly 0.23 m ahead of the axle (owner); map_server fallback 0.23.
stereo_camera_optical y -0.041: the vendor ESKF base_vio (0.466, -0.041, drive-axle origin)
puts the optical centre on the right eye; it feeds the costmap, collision monitor and the
non-grass projector. mower_sim gps_antenna_x 0.098; tests follow.

File: config/urdf/mower.urdf.xacro (robot description, xacro)
@@ -37,7 +37,8 @@
               arm — without it, it silently assumes the receiver sits
               at the robot origin.
-              Offset: x +0.10 measured by the owner 2026-10-20 (antenna
-              centre 0.10 m ahead of the rear axle, centred left-right);
-              z +0.30 vendor. Before it was (0, 0, 0.3) and navsat put
+              Offset (0.098, 0, 0.214): the vendor ESKF base_gps_x 0.098
+              (CAD, drive-axle origin; the owner measured 0.10, centred)
+              and the antenna top 0.214 m above the wheel axle (vendor
+              eskf cfg.yaml). Was (0, 0, 0.3). Before it was (0, 0, 0.3) and navsat put
               base_link at the antenna: the field pivot test saw a 7-10 cm
               /fix circle and 0.08-0.19 m of EKF "displacement" per pivot
@@ -98,10 +99,10 @@
        identity broadcast (see the frame contract above). -->
   <xacro:property name="imu_xyz"    value="0 0 0"/>
-  <xacro:property name="gps_xyz"    value="0.10 0 0.3"/>
+  <xacro:property name="gps_xyz"    value="0.098 0 0.214"/>
   <xacro:property name="bumper_xyz" value="0.50718 0 0"/>
-  <!-- cutter_xyz x 0.25 (was 0.3): the owner measured the deck centre 0.25 m ahead of the
-       rear axle, centred (2026-10-20). cutter_link and blade_link share it; map_server's mow
-       progress looks up base_link -> blade_link (fallback blade_offset_x, also 0.25). -->
-  <xacro:property name="cutter_xyz" value="0.25 0 -0.05"/>
+  <!-- cutter_xyz x 0.23 (was 0.3): the owner measured the deck centre exactly 0.23 m ahead
+       of the rear axle, centred (2026-10-20). cutter_link and blade_link share it; map_server's mow
+       progress looks up base_link -> blade_link (fallback blade_offset_x, also 0.23). -->
+  <xacro:property name="cutter_xyz" value="0.23 0 -0.05"/>
   <!-- Cutter disc radius: 0.20 m cut width. TODO: measure the blade tip circle on the
        Tron and update this, the coverage cut_width_m launch arg (mower.launch.py) and
@@ -223,5 +224,5 @@
        broadcast (see frame contract). TODO(calib): real offset here. -->
   <xacro:box_sensor name="imu_link" xyz="${imu_xyz}" rpy="0 0 0" size="${sensor_box}" material="green"/>
-  <!-- GNSS antenna (UM960): measured lever arm (x 0.10, owner 2026-10-20). -->
+  <!-- GNSS antenna (UM960): vendor CAD lever arm x 0.098 (owner measured 0.10), z 0.214. -->
   <xacro:box_sensor name="gps_link" xyz="${gps_xyz}" rpy="0 0 0" size="${sensor_box}" material="red"/>
   <!-- Bumper strip. -->
@@ -245,5 +246,7 @@
     <parent link="base_link"/>
     <child link="stereo_camera_optical"/>
-    <origin xyz="0.466 0 0.240" rpy="-1.5547956 0 -1.5707963"/>
+    <!-- y -0.041 (was 0, 2026-10-20): the vendor ESKF base_vio (0.466, -0.041), drive-axle
+         origin, puts the optical centre on the RIGHT eye (the disparity reference). -->
+    <origin xyz="0.466 -0.041 0.240" rpy="-1.5547956 0 -1.5707963"/>
   </joint>
   <!-- Metoak stereo IMU (ICM-40608 on i2c 8-0068; mower_cameras/stereo_imu -> /stereo_imu/data,

Commit message: geometry: owner-measured footprint and the MCU's 0.40 m wheel split
Owner measured (2026-10-20, from the rear axle = base_link): tyre track 0.39 m,
tyres 0.22 m / 6 cm, bumper +0.60, rear -0.10, 0.47 m wide with the wheel trim.
The field pivot bag gives IMU / MCU-reported yaw rate 1.02-1.03 on clean pivots,
i.e. the MCU splits (v, w) with b ~0.40 (vendor wheel_base 0.4, WHEELBASE_M 0.40),
not the stale vendor URDF 0.48.

- wheel-speed math b 0.48 -> 0.40 everywhere (cmd_vel_slew, WheelFloorCritic x3,
  docking, hard boundary, sim split, gate evaluator, bag metrics)
- pivot floor 0.06 / 0.20 = 0.3 rad/s = the MCU clamp: Spin min = max = 0.3, and
  cmd_vel_slew steps a pure rotation straight to the floor or to 0 (pivot_floor_step)
- tightest arc at |w| 0.3: v 0.12, r 0.40 (was 0.132 / 0.44); coverage clamp 0.40
- footprint [[0.60, 0.235], [0.60, -0.235], [-0.10, -0.235], [-0.10, 0.235]] in
  both costmaps, collision_monitor zones moved with the nose (same bands), FTC,
  mission obstacle footprint, path conditioning, rear guard, sim world
- global inflation 0.70 / 6.5 (circumscribed 0.67, inscribed now 0.12)
- URDF wheels: radius 0.11, width 0.06, axle x 0, track y 0.195; chassis box
- mower_sim: ground track 0.39 (pivots turn 2.6 % faster than commanded)

File: config/urdf/mower.urdf.xacro (robot description, xacro)
@@ -76,11 +76,17 @@
   <!-- Chassis visual box (cosmetic; the base_link origin stays at the
        rear drive axle centre regardless of where the box is drawn). -->
-  <xacro:property name="chassis_size" value="0.7 0.5 0.2"/>
-  <xacro:property name="chassis_xyz"  value="0.12 0 0"/>
-  <!-- Wheels (vendor values). Drive axle x, track half-width y, drop z. -->
-  <xacro:property name="wheel_radius"  value="0.1"/>
-  <xacro:property name="wheel_width"   value="0.05"/>
-  <xacro:property name="drive_axle_x"  value="-0.098"/>
-  <xacro:property name="drive_track_y" value="0.24"/>
+  <!-- Owner-measured 2026-10-20 from the rear axle: rear -0.10, front bumper +0.60, 0.46 m
+       wide (0.47 with the wheel trim) -> 0.70 x 0.46 box centred at x=+0.25 (was 0.7 x 0.5 at
+       +0.12, vendor). The nav2 footprint is the same outline (nav2_params.yaml). -->
+  <xacro:property name="chassis_size" value="0.7 0.46 0.2"/>
+  <xacro:property name="chassis_xyz"  value="0.25 0 0"/>
+  <!-- Wheels, owner-measured 2026-10-20 (were the stale vendor 0.1 / 0.05 / -0.098 / 0.24):
+       tyre diameter 0.22, tread 0.06, tyre centre-to-centre track 0.39 (half 0.195); the
+       drive axle IS base_link (x 0). The MCU splits (v, w) with b 0.40 (cmd_vel_slew
+       TRACK_WIDTH_M), not with this physical track. Drop z unchanged (cosmetic). -->
+  <xacro:property name="wheel_radius"  value="0.11"/>
+  <xacro:property name="wheel_width"   value="0.06"/>
+  <xacro:property name="drive_axle_x"  value="0.0"/>
+  <xacro:property name="drive_track_y" value="0.195"/>
   <xacro:property name="wheel_drop_z"  value="-0.05"/>
   <!-- Omni wheels (castor pair at the front), canted by omni_yaw about Z. -->

Commit message: urdf: bumper at the owner-measured front (face at 0.60, 0.46 wide); visual only

File: config/urdf/mower.urdf.xacro (robot description, xacro)
@@ -106,5 +106,5 @@
   <xacro:property name="imu_xyz"    value="0 0 0"/>
   <xacro:property name="gps_xyz"    value="0.098 0 0.214"/>
-  <xacro:property name="bumper_xyz" value="0.50718 0 0"/>
+  <xacro:property name="bumper_xyz" value="0.59 0 0"/>  <!-- front face at the owner-measured 0.60 -->
   <!-- cutter_xyz x 0.23 (was 0.3): the owner measured the deck centre exactly 0.23 m ahead
        of the rear axle, centred (2026-10-20). cutter_link and blade_link share it; map_server's mow
@@ -120,5 +120,5 @@
   <xacro:property name="rear_cam_xyz"   value="-0.201 0 0.25"/>
   <xacro:property name="sensor_box" value="0.05 0.05 0.05"/>
-  <xacro:property name="bumper_box" value="0.02 0.5 0.1"/>
+  <xacro:property name="bumper_box" value="0.02 0.46 0.1"/>
   <!-- ============================ macros ============================ -->
   <!-- Fixed box sensor on a fixed joint off base_link.
